File: Eagle/rev1/MA163.sch (EAGLE design)
At the start: 46 parts, among them IC1 Z80, IC10 74LS157N, IC11 74LS374N, IC12 74LS374N, IC13 4416, IC14 4416, IC2 2764, IC3 2764, IC4 74LS00N, IC5 74LS32N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

Commit message: Preparado board para roteamento
Parts:
- added RN1: (no value), resistor-net:RN10
- R10, R11, R12, R13, R14, R15, R16, R17, R8, R9: device rcl:R-EU_0207/5V -> rcl:R-EU_0207/2V
- R7: device rcl:R-EU_0207/10 -> rcl:R-EU_0207/12
Connections:
- net LPT_!ACK: now also RN1.2
- net LPT_!STROBE: now also RN1.3
- net LPT_D0: now also RN1.4
- net LPT_D1: now also RN1.5
- net LPT_D2: now also RN1.6
- net LPT_D3: now also RN1.7
- net LPT_D4: now also RN1.8
- net LPT_D5: now also RN1.9
- net LPT_D6: now also RN1.10
- net LPT_D7: now also RN1.11
- net VCC: now also RN1.1
Other:
- note added: "Microdigital Parallel Card"
- note removed: "Microdigital MA163"
- moved on the sheet: IC7B, LPT, R10, R11, R12, R13, R14, R15, R16, R17, R2, R8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

Commit message: wip
Connections:
- net LPT_!ACK: now also RN1.11; no longer RN1.2
- net LPT_!STROBE: now also RN1.10; no longer RN1.3
- net LPT_D0: now also RN1.9; no longer RN1.4
- net LPT_D1: now also RN1.8; no longer RN1.5
- net LPT_D2: now also RN1.7; no longer RN1.6
- net LPT_D3: now also RN1.6; no longer RN1.7
- net LPT_D4: now also RN1.5; no longer RN1.8
- net LPT_D5: now also RN1.4; no longer RN1.9
- net LPT_D6: now also RN1.3; no longer RN1.10
- net LPT_D7: now also RN1.2; no longer RN1.11
Other:
- moved on the sheet: RN1
Changed lines of the file:
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@@
 <attribute name="VALUE" x="17.78" y="81.28" size="1.778" layer="96" rot="R90"/>
 </instance>
-<instance part="RN1" gate="1" x="15.24" y="22.86" smashed="yes">
-<attribute name="NAME" x="12.7" y="25.146" size="1.778" layer="95"/>
-<attribute name="VALUE" x="12.7" y="18.796" size="1.778" layer="96"/>
+<instance part="RN1" gate="1" x="71.12" y="22.86" smashed="yes" rot="R180">
+<attribute name="NAME" x="73.66" y="20.574" size="1.778" layer="95" rot="R180"/>
+<attribute name="VALUE" x="73.66" y="26.924" size="1.778" layer="96" rot="R180"/>
 </instance>
-<instance part="P+14" gate="VCC" x="7.62" y="27.94" smashed="yes">
-<attribute name="VALUE" x="5.08" y="25.4" size="1.778" layer="96" rot="R90"/>
+<instance part="P+14" gate="VCC" x="81.28" y="22.86" smashed="yes" rot="R270">
+<attribute name="VALUE" x="78.74" y="25.4" size="1.778" layer="96"/>
 </instance>
 </instances>
@@
 <pinref part="P+14" gate="VCC" pin="VCC"/>
 <pinref part="RN1" gate="1" pin="1"/>
-<wire x1="7.62" y1="25.4" x2="7.62" y2="22.86" width="0.1524" layer="91"/>
-<wire x1="7.62" y1="22.86" x2="10.16" y2="22.86" width="0.1524" layer="91"/>
+<wire x1="78.74" y1="22.86" x2="76.2" y2="22.86" width="0.1524" layer="91"/>
 </segment>
 </net>
@@
 <wire x1="25.4" y1="66.04" x2="25.4" y2="58.42" width="0.1524" layer="91"/>
 <junction x="25.4" y="58.42"/>
-<pinref part="RN1" gate="1" pin="3"/>
+<pinref part="RN1" gate="1" pin="10"/>
 <wire x1="25.4" y1="22.86" x2="25.4" y2="58.42" width="0.1524" layer="91"/>
 </segment>
@@
 <wire x1="20.32" y1="60.96" x2="20.32" y2="35.56" width="0.1524" layer="91"/>
 <junction x="20.32" y="35.56"/>
-<pinref part="RN1" gate="1" pin="2"/>
+<pinref part="RN1" gate="1" pin="11"/>
 <wire x1="20.32" y1="22.86" x2="20.32" y2="35.56" width="0.1524" layer="91"/>
 </segment>
@@
 <wire x1="30.48" y1="60.96" x2="30.48" y2="55.88" width="0.1524" layer="91"/>
 <junction x="30.48" y="55.88"/>
-<pinref part="RN1" gate="1" pin="4"/>
+<pinref part="RN1" gate="1" pin="9"/>
 <wire x1="30.48" y1="22.86" x2="30.48" y2="55.88" width="0.1524" layer="91"/>
 </segment>
@@
 <wire x1="35.56" y1="66.04" x2="35.56" y2="53.34" width="0.1524" layer="91"/>
 <junction x="35.56" y="53.34"/>
-<pinref part="RN1" gate="1" pin="5"/>
+<pinref part="RN1" gate="1" pin="8"/>
 <wire x1="35.56" y1="22.86" x2="35.56" y2="53.34" width="0.1524" layer="91"/>
 </segment>
@@
 <wire x1="40.64" y1="60.96" x2="40.64" y2="50.8" width="0.1524" layer="91"/>
 <junction x="40.64" y="50.8"/>
-<pinref part="RN1" gate="1" pin="6"/>
+<pinref part="RN1" gate="1" pin="7"/>
 <wire x1="40.64" y1="22.86" x2="40.64" y2="50.8" width="0.1524" layer="91"/>
 </segment>
@@
 <wire x1="45.72" y1="66.04" x2="45.72" y2="48.26" width="0.1524" layer="91"/>
 <junction x="45.72" y="48.26"/>
-<pinref part="RN1" gate="1" pin="7"/>
+<pinref part="RN1" gate="1" pin="6"/>
 <wire x1="45.72" y1="22.86" x2="45.72" y2="48.26" width="0.1524" layer="91"/>
 </segment>
@@
 <wire x1="50.8" y1="60.96" x2="50.8" y2="45.72" width="0.1524" layer="91"/>
 <junction x="50.8" y="45.72"/>
-<pinref part="RN1" gate="1" pin="8"/>
+<pinref part="RN1" gate="1" pin="5"/>
 <wire x1="50.8" y1="22.86" x2="50.8" y2="45.72" width="0.1524" layer="91"/>
 </segment>
@@
 <wire x1="55.88" y1="66.04" x2="55.88" y2="43.18" width="0.1524" layer="91"/>
 <junction x="55.88" y="43.18"/>
-<pinref part="RN1" gate="1" pin="9"/>
+<pinref part="RN1" gate="1" pin="4"/>
 <wire x1="55.88" y1="22.86" x2="55.88" y2="43.18" width="0.1524" layer="91"/>
 </segment>
@@
 <wire x1="60.96" y1="60.96" x2="60.96" y2="40.64" width="0.1524" layer="91"/>
 <junction x="60.96" y="40.64"/>
-<pinref part="RN1" gate="1" pin="10"/>
+<pinref part="RN1" gate="1" pin="3"/>
 <wire x1="60.96" y1="22.86" x2="60.96" y2="40.64" width="0.1524" layer="91"/>
 </segment>
@@
 <wire x1="66.04" y1="66.04" x2="66.04" y2="38.1" width="0.1524" layer="91"/>
 <junction x="66.04" y="38.1"/>
-<pinref part="RN1" gate="1" pin="11"/>
+<pinref part="RN1" gate="1" pin="2"/>
 <wire x1="66.04" y1="22.86" x2="66.04" y2="38.1" width="0.1524" layer="91"/>
 </segment>
