File: Eagle/rev1/MA163.brd (EAGLE design)
At the start: 127 x 82.5 mm, 47 parts, among them IC1 Z80, IC10 74LS157N, IC11 74LS374N, IC12 74LS374N, IC13 4416, IC14 4416, IC2 2764, IC3 2764, IC4 74LS00N, IC5 74LS32N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

Commit message: Roteando
Parts:
- moved IC11 12.7 mm to (106.7, 34.9)
- moved IC12 12.7 mm to (106.7, 22.2)
- turned LPT to 270 degrees
- turned R5 to 90 degrees
- turned R6 to 90 degrees
Routing:
- net VCC: track 0.00 -> 444.9 mm, vias 0 -> 5
- net GND: track 0.00 -> 121.5 mm, vias 0 -> 3
- net A0: track 0.00 -> 43.7 mm
- net !IOSEL: track 0.00 -> 42.1 mm, vias 0 -> 2
- net Z80_D5: track 0.00 -> 31.0 mm
- net N$14: track 0.00 -> 11.4 mm, vias 0 -> 1
- added copper zone on layer 1, net GND
- added copper zone on layer 16, net GND
Other:
- outline, holes or cut-outs redrawn

Commit message: Mais roteamento
Routing:
- net D2: track 0.00 -> 77.9 mm, vias 0 -> 1
- net D1: track 0.00 -> 70.7 mm, vias 0 -> 1
- net D0: track 0.00 -> 69.2 mm
- net A1: track 0.00 -> 34.8 mm
- net A2: track 0.00 -> 34.6 mm
- net A3: track 0.00 -> 33.0 mm
- net A7: track 0.00 -> 33.0 mm
- net A5: track 0.00 -> 33.0 mm
- net A4: track 0.00 -> 33.0 mm
- net A6: track 0.00 -> 27.2 mm, vias 0 -> 1
- net !RESET: track 0.00 -> 8.18 mm, vias 0 -> 1
- net !DEVSEL: track 0.00 -> 5.81 mm, vias 0 -> 1
- net PHASE0: track 0.00 -> 5.69 mm, vias 0 -> 1
- net Q3: track 0.00 -> 5.56 mm, vias 0 -> 1
- net N$1: track 0.00 -> 5.08 mm
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
Commit message: wip
Parts:
- moved R2 0.45 mm to (22.9, 51.8), turned to 90 degrees
- turned R1 to 0 degrees
Routing:
- net !WR: track 0.00 -> 184.8 mm, vias 0 -> 2
- net !MREQ: track 0.00 -> 146.6 mm, vias 0 -> 4
- net !RD: track 0.00 -> 88.7 mm, vias 0 -> 1
- net Z80_D6: track 0.00 -> 84.0 mm, vias 0 -> 4
- net MEM_A4: track 0.00 -> 74.3 mm, vias 0 -> 1
- net MEM_A5: track 0.00 -> 60.6 mm, vias 0 -> 3
- net Z80_D7: track 0.00 -> 55.2 mm, vias 0 -> 2
- net MEM_A6: track 0.00 -> 45.0 mm
- net GND: vias 4 -> 5

Commit message: wip
Parts:
- moved R10 2.54 mm to (100.3, 45.1)
- moved R11 2.54 mm to (102.9, 45.1)
- moved R12 2.54 mm to (105.4, 45.1)
- moved R13 2.54 mm to (108.0, 45.1)
- moved R14 2.54 mm to (110.5, 45.1)
- moved R15 2.54 mm to (113.0, 45.1)
- moved R16 2.54 mm to (115.6, 45.1)
- moved R17 2.54 mm to (118.1, 45.1)
- moved R8 2.54 mm to (95.2, 45.1)
- moved R9 2.54 mm to (97.8, 45.1)
Connections:
- net LPT_!ACK: now also RN1.11; no longer RN1.2
- net LPT_!STROBE: now also RN1.10; no longer RN1.3
- net LPT_D0: now also RN1.9; no longer RN1.4
- net LPT_D1: now also RN1.8; no longer RN1.5
- net LPT_D2: now also RN1.7; no longer RN1.6
- net LPT_D3: now also RN1.6; no longer RN1.7
- net LPT_D4: now also RN1.5; no longer RN1.8
- net LPT_D5: now also RN1.4; no longer RN1.9
- net LPT_D6: now also RN1.3; no longer RN1.10
- net LPT_D7: now also RN1.2; no longer RN1.11
Routing:
- net LPT_!STROBE: track 0.00 -> 161.2 mm, vias 0 -> 1
- net Z80_A11: track 0.00 -> 139.4 mm, vias 0 -> 4
- net !DEVSEL: track 5.81 -> 122.6 mm, vias 1 -> 3
- net N$1: track 5.08 -> 68.5 mm, vias 0 -> 1
- net Z80_D4: track 0.00 -> 41.6 mm, vias 0 -> 1
- net Z80_D5: track 31.0 -> 70.8 mm, vias 0 -> 2
- net LPT_D0: track 0.00 -> 38.3 mm
- net LPT_D1: track 0.00 -> 33.2 mm
- net LPT_D2: track 0.00 -> 29.6 mm
- net VCC: track 444.9 -> 471.3 mm
- net LPT_D3: track 0.00 -> 26.0 mm
- net FLAG_FW: track 0.00 -> 22.6 mm
- net LPT_D4: track 0.00 -> 22.4 mm
- net LPT_D5: track 0.00 -> 19.9 mm
- net LPT_D6: track 0.00 -> 17.9 mm
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
Commit message: wip
Routing:
- net !RESET: track 8.18 -> 212.0 mm, vias 1 -> 4
- net LPT_LATCH: track 0.00 -> 198.4 mm, vias 0 -> 1
- net Q3: track 5.56 -> 194.7 mm, vias 1 -> 3
- net BUS_RD: track 0.00 -> 181.3 mm
- net LPT_!ACK: track 0.00 -> 172.6 mm, vias 0 -> 5
- net ROM!CE: track 0.00 -> 145.0 mm, vias 0 -> 2
- net Z80_D6: track 84.0 -> 225.3 mm, vias 4 -> 5
- net !Z80_CLK: track 0.00 -> 139.6 mm, vias 0 -> 3
- net Z80_D5: track 70.8 -> 206.6 mm, vias 2 -> 4
- net Z80_D3: track 0.00 -> 116.8 mm, vias 0 -> 2
- net Z80_D7: track 55.2 -> 167.6 mm, vias 2 -> 3
- net Z80_A14: track 0.00 -> 112.2 mm, vias 0 -> 1
- net Z80_D2: track 0.00 -> 109.1 mm, vias 0 -> 1
- net Z80_A15: track 0.00 -> 108.5 mm, vias 0 -> 1
- net Z80_A9: track 0.00 -> 101.7 mm, vias 0 -> 3
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
Commit message: Roteamento finalizado
Parts:
- turned R4 to 270 degrees
Routing:
- net Z80_A12: track 8.89 -> 134.8 mm, vias 1 -> 3
- net Z80_A4: track 13.3 -> 84.6 mm, vias 0 -> 2
- net Z80_D2: track 109.1 -> 174.3 mm, vias 1 -> 2
- net MEM_A7: track 0.00 -> 59.1 mm, vias 0 -> 1
- net Z80_A6: track 13.3 -> 70.0 mm, vias 0 -> 2
- net Z80_A7: track 13.3 -> 68.6 mm
- net MEM_A3: track 0.00 -> 48.9 mm, vias 0 -> 1
- net Z80_A3: track 13.3 -> 61.6 mm
- net Z80_D4: track 114.7 -> 162.5 mm
- net Z80_D0: track 91.5 -> 137.8 mm, vias 1 -> 2
- net FF_HIGH32K: track 0.00 -> 45.3 mm, vias 0 -> 2
- net Z80_D1: track 97.9 -> 139.0 mm, vias 1 -> 2
- net Z80_A10: track 65.5 -> 105.4 mm
- net Z80_A1: track 13.3 -> 52.2 mm, vias 0 -> 1
- net Z80_A0: track 13.3 -> 52.1 mm
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Other:
- outline, holes or cut-outs redrawn
